File: Hardware/CAN_Gauge.kicad_pcb (KiCad board)
At the start: 2 copper layers, 50 x 50 mm, 77 parts, among them J1 Conn_02x03_Odd_Even, J2 Conn_01x08, SW1 SW_Push, U1 STM32F103C8Tx, U2 SN65HVD230, U3 2594, U4 UG-2864HSWEG01

Commit message: Work in progress
Parts:
- moved R17 2.89 mm to (141.1, 75.4)
- moved R18 2.89 mm to (137.9, 75.4)
- moved R21 2.89 mm to (134.6, 75.4)
- moved R16 2.89 mm to (139.5, 75.4)
- moved R19 2.89 mm to (136.2, 75.4)
Routing:
- net GND: track 84.2 -> 80.7 mm, vias 29 -> 30
- net Net-(D4-Pad2): track 7.21 -> 4.87 mm
- net Net-(D7-Pad2): track 14.7 -> 16.8 mm
- net LED4: track 3.56 -> 5.64 mm
- net Net-(D8-Pad2): track 24.7 -> 26.8 mm
- net Net-(D5-Pad2): track 4.59 -> 2.97 mm
- net Net-(D6-Pad2): track 8.72 -> 10.3 mm
- net /STM/CONFIG_1: track 11.3 -> 9.89 mm
- net LED5: track 4.03 -> 5.33 mm
- net OSC_IN: track 0.00 -> 0.80 mm
- net LED8: track 7.20 -> 6.54 mm
- net LED7: track 6.14 -> 5.62 mm
Other:
- board text added: "CAN Gauge F103 RevA"
- board text removed: "CAN Gauge 103_A"

Commit message: Update pcb
Connections:
- net Net-(U1-Pad21) renamed /STM/CONFIG_4
- net Net-(U1-Pad22) renamed /STM/CONFIG_5
Routing:
- net +3V3: track 19.2 -> 22.4 mm
- net OSC_IN: track 0.80 -> 0.00 mm
