File: Hardware/CAN_Gauge.kicad_pcb (KiCad board)
At the start: 2 copper layers, 50 x 50 mm, 77 parts, among them J1 Conn_02x03_Odd_Even, J2 Conn_01x08, SW1 SW_Push, U1 STM32F103C8Tx, U2 SN65HVD230, U3 2594, U4 UG-2864HSWEG01

Commit message: Update PCB
Parts:
- added C6: 0.1u, Capacitor_SMD:C_0402_1005Metric, F.Cu at (142.6, 89.3)
- moved R1 0.69 mm to (137.9, 91.7)
Connections:
- net Net-(U1-Pad20) renamed /STM/CONFIG_3
Routing:
- net GND: track 80.7 -> 73.9 mm, vias 30 -> 31
- net NRST: track 25.1 -> 28.5 mm
- net +3V3: track 22.4 -> 20.8 mm
- net Net-(D2-Pad2): track 19.5 -> 18.1 mm
- net LED9: track 28.2 -> 27.0 mm
- net Net-(D10-Pad2): track 7.37 -> 6.19 mm
- net BOOT0: track 3.77 -> 2.96 mm
- net Net-(D1-Pad2): track 27.8 -> 27.0 mm

Commit message: PCB updates, Generate Gerbers, BOM, and position files
Parts:
- added C12: 0.1u, Capacitor_SMD:C_0402_1005Metric, F.Cu at (119.9, 80.5)
- added JP4: SolderJumper_2_Open, Jumper:SolderJumper-2_P1.3mm_Open_Pad1.0x1.5mm, F.Cu at (125.4, 78.1)
- added JP5: SolderJumper_2_Open, Jumper:SolderJumper-2_P1.3mm_Open_Pad1.0x1.5mm, F.Cu at (126.0, 80.6)
- added JP6: SolderJumper_2_Open, Jumper:SolderJumper-2_P1.3mm_Open_Pad1.0x1.5mm, F.Cu at (126.7, 83.2)
Connections:
- U1 pad 20: /STM/CONFIG_3 -> Net-(U1-Pad20)
- U1 pad 21: /STM/CONFIG_4 -> Net-(U1-Pad21)
- U1 pad 22: /STM/CONFIG_5 -> Net-(U1-Pad22)
- U1 pad 26: Net-(U1-Pad26) -> /STM/CONFIG_3
- U1 pad 27: Net-(U1-Pad27) -> /STM/CONFIG_4
- U1 pad 28: Net-(U1-Pad28) -> /STM/CONFIG_5
Routing:
- net GND: track 73.9 -> 83.4 mm, vias 31 -> 32
- net /STM/CONFIG_3: track 0.00 -> 8.51 mm
- net /STM/CONFIG_4: track 0.00 -> 6.40 mm
- net /STM/CONFIG_5: track 0.00 -> 4.91 mm
- net NRST: track 28.5 -> 30.9 mm
- net /STM/CONFIG_2: track 14.9 -> 14.4 mm
Other:
- board text added: "3"
- board text added: "4"
- board text added: "5"
- board text added: "Gauge F103 RevA"
- board text removed: "CAN Gauge F103 RevA"
