File: Hardware/OLED.sch (KiCad schematic (older format))
At the start: 9 parts, among them U4 UG-2864HSWEG01

Commit message: Update components for assembly, generate gerbers
Parts:
- C16: Comments (none) -> X5R 2.2uF ±10% 10V 0402 Multilayer Ceramic Capacitors MLCC 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; LCSC (none) -> C77002
- C18: Field5 (none) -> X5R 2.2uF ±10% 10V 0402 Multilayer Ceramic Capacitors MLCC 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; LCSC (none) -> C77002
Changed lines of the file:
@@
 F 2 "Capacitor_SMD:C_0402_1005Metric" H 4748 2550 50  0001 C CNN
 F 3 "~" H 4710 2700 50  0001 C CNN
+F 4 "C77002" V 4710 2700 50  0001 C CNN "LCSC"
+F 5 "X5R 2.2uF ±10% 10V 0402 Multilayer Ceramic Capacitors MLCC - SMD/SMT ROHS" V 4710 2700 50  0001 C CNN "Comments"
 	1    4710 2700
 	0    -1   -1   0
@@
 F 2 "Capacitor_SMD:C_0402_1005Metric" H 4888 2350 50  0001 C CNN
 F 3 "~" H 4850 2500 50  0001 C CNN
+F 4 "C77002" V 4850 2500 50  0001 C CNN "LCSC"
+F 5 "X5R 2.2uF ±10% 10V 0402 Multilayer Ceramic Capacitors MLCC - SMD/SMT ROHS" V 4850 2500 50  0001 C CNN "Field5"
 	1    4850 2500
 	0    -1   -1   0

Commit message: Update board layout
Fix OLED pads to meet intended design. Move all non UI components to one side of the board for better single sided assembly.
Parts:
- added TP6: TestPoint, TestPoint:TestPoint_Pad_D1.0mm, symbol Connector:TestPoint
Connections:
- wire segments 76 -> 78
Changed lines of the file:
@@
 Text Label 4960 3700 0    50   ~ 0
 RST
-$Comp
-L power:+3.3V #PWR0158
-U 1 1 61BD266D
-P 3760 4400
-F 0 "#PWR0158" H 3760 4250 50  0001 C CNN
-F 1 "+3.3V" H 3775 4573 50  0000 C CNN
-F 2 "" H 3760 4400 50  0001 C CNN
-F 3 "" H 3760 4400 50  0001 C CNN
-	1    3760 4400
-	1    0    0    -1
-$EndComp
 Wire Wire Line
 	5240 4800 5090 4800
-Wire Wire Line
-	5090 4800 5090 4700
 Connection ~ 5090 4700
 Wire Wire Line
 	5240 4700 5090 4700
-Wire Wire Line
-	5090 4700 5090 4600
 Wire Wire Line
 	5090 4600 5090 4500
@@
 Wire Wire Line
 	5090 4400 5090 4500
-Connection ~ 5090 4400
 Wire Wire Line
 	5240 4400 5090 4400
@@
 I2C1_SDA
 Wire Wire Line
-	3760 4400 5090 4400
+	5090 4700 5090 4800
+$Comp
+L Connector:TestPoint TP?
+U 1 1 61BB6AF7
+P 4320 4560
+AR Path="/615E5281/61BB6AF7" Ref="TP?"  Part="1"
+AR Path="/615E7CAC/61BB6AF7" Ref="TP?"  Part="1"
+AR Path="/615E795E/61BB6AF7" Ref="TP6"  Part="1"
+F 0 "TP6" H 4378 4678 50  0000 L CNN
+F 1 "TestPoint" H 4378 4587 50  0000 L CNN
+F 2 "TestPoint:TestPoint_Pad_D1.0mm" H 4520 4560 50  0001 C CNN
+F 3 "~" H 4520 4560 50  0001 C CNN
+	1    4320 4560
+	1    0    0    -1
+$EndComp
+Wire Wire Line
+	4320 4560 4320 4640
+Wire Wire Line
+	4320 4640 5090 4640
+Wire Wire Line
+	5090 4600 5090 4640
+Connection ~ 5090 4640
+Wire Wire Line
+	5090 4640 5090 4700
 $EndSCHEMATC

Commit message: Updates
Parts:
- C13: value 1u -> 0.1u; LCSC (none) -> C1525
- C14, C15, C17: LCSC (none) -> C52923
- C16, C18: LCSC C77002 -> C170151
- R26: LCSC (none) -> C25744
Changed lines of the file:
@@
 Title "CAN Gauge"
 Date "2021-10-10"
-Rev "B"
+Rev "C"
 Comp ""
 Comment1 ""
@@
 F 2 "Resistor_SMD:R_0402_1005Metric" V 4050 5310 50  0001 C CNN
 F 3 "~" H 4010 5320 50  0001 C CNN
+F 4 " C25744" H 4010 5320 50  0001 C CNN "LCSC"
 	1    4010 5320
 	-1   0    0    1
@@
 F 2 "Capacitor_SMD:C_0402_1005Metric" H 4408 5160 50  0001 C CNN
 F 3 "~" H 4370 5310 50  0001 C CNN
+F 4 " C52923" H 4370 5310 50  0001 C CNN "LCSC"
 	1    4370 5310
 	-1   0    0    1
@@
 F 2 "Capacitor_SMD:C_0402_1005Metric" H 4768 5150 50  0001 C CNN
 F 3 "~" H 4730 5300 50  0001 C CNN
+F 4 " C52923" H 4730 5300 50  0001 C CNN "LCSC"
 	1    4730 5300
 	-1   0    0    1
@@
 P 3800 3050
 F 0 "C13" H 3685 3004 50  0000 R CNN
-F 1 "1u" H 3685 3095 50  0000 R CNN
+F 1 "0.1u" H 3685 3095 50  0000 R CNN
 F 2 "Capacitor_SMD:C_0402_1005Metric" H 3838 2900 50  0001 C CNN
 F 3 "~" H 3800 3050 50  0001 C CNN
+F 4 "C1525" H 3800 3050 50  0001 C CNN "LCSC"
 	1    3800 3050
 	-1   0    0    1
@@
 F 2 "Capacitor_SMD:C_0402_1005Metric" H 4098 3200 50  0001 C CNN
 F 3 "~" H 4060 3350 50  0001 C CNN
+F 4 " C52923" H 4060 3350 50  0001 C CNN "LCSC"
 	1    4060 3350
 	-1   0    0    1
@@
 F 2 "Capacitor_SMD:C_0402_1005Metric" H 4748 2550 50  0001 C CNN
 F 3 "~" H 4710 2700 50  0001 C CNN
-F 4 "C77002" V 4710 2700 50  0001 C CNN "LCSC"
+F 4 " C170151" V 4710 2700 50  0001 C CNN "LCSC"
 F 5 "X5R 2.2uF ±10% 10V 0402 Multilayer Ceramic Capacitors MLCC - SMD/SMT ROHS" V 4710 2700 50  0001 C CNN "Comments"
 	1    4710 2700
@@
 F 2 "Capacitor_SMD:C_0402_1005Metric" H 4888 2350 50  0001 C CNN
 F 3 "~" H 4850 2500 50  0001 C CNN
-F 4 "C77002" V 4850 2500 50  0001 C CNN "LCSC"
+F 4 " C170151" V 4850 2500 50  0001 C CNN "LCSC"
 F 5 "X5R 2.2uF ±10% 10V 0402 Multilayer Ceramic Capacitors MLCC - SMD/SMT ROHS" V 4850 2500 50  0001 C CNN "Field5"
 	1    4850 2500

Commit message: Generate files
Parts:
- U4: footprint custom:SSH1106_Bottom -> custom:SSD1306_FFC; LCSC (none) -> C2797216
Changed lines of the file:
@@
 U 1 1 6158C49D
 P 4790 5500
+AR Path="/615E795E/6158C49D" Ref="U4"  Part="1"
+AR Path="/615E5281/6158C49D" Ref="U4"  Part="1"
 F 0 "U4" H 6218 7196 50  0000 L CNN
 F 1 "UG-2864HSWEG01" H 6218 7105 50  0000 L CNN
-F 2 "custom:SSH1106_Bottom" H 5440 8750 50  0001 C CNN
+F 2 "custom:SSD1306_FFC" H 5440 8750 50  0001 C CNN
 F 3 "" H 5440 8750 50  0001 C CNN
+F 4 "C2797216 " H 4790 5500 50  0001 C CNN "LCSC"
 	1    4790 5500
 	1    0    0    -1

Commit message: Update PCB
Parts:
- U4: footprint custom:SSD1306_FFC -> custom:SSH1106_Bottom
Changed lines of the file:
@@
 F 0 "U4" H 6218 7196 50  0000 L CNN
 F 1 "UG-2864HSWEG01" H 6218 7105 50  0000 L CNN
-F 2 "custom:SSD1306_FFC" H 5440 8750 50  0001 C CNN
+F 2 "custom:SSH1106_Bottom" H 5440 8750 50  0001 C CNN
 F 3 "" H 5440 8750 50  0001 C CNN
 F 4 "C2797216 " H 4790 5500 50  0001 C CNN "LCSC"
